File: simulations/power_amplifiers/classAB_simul/classAB_simul.sch (KiCad schematic (older format))
At the start: 5 parts

Commit message: more simulation schematic
Parts:
- added C? (x2): C, symbol pspice:C
- added L?: INDUCTOR, symbol pspice:INDUCTOR
- added R? (x3): R, symbol pspice:R
- added R? (x2): 100k, symbol pspice:R
- added U?: TL081, symbol Amplifier_Operational:TL081
- added V? (x2): VSOURCE, symbol pspice:VSOURCE
- D? (x2): value DIODE -> 1N4148
- Q?: value QNPN -> BD135
- Q?: value QPNP -> BD136
Connections:
- net labels added: input
- wire segments 10 -> 44
- no-connect marks 0 -> 4
Other:
- note added: "headphones / speaker"

Commit message: update simulation
Parts:
- removed D? (x2): 1N4148, symbol pspice:DIODE
- added D1, D2: 1N4148, symbol pspice:DIODE
- 230u1: renamed from L?; Spice_Model (none) -> 230u; Spice_Netlist_Enabled (none) -> Y; Spice_Primitive (none) -> L
- C1: renamed from C?; value C -> 2.2uF
- C2: renamed from C?; value C -> 100u
- Q1: renamed from Q?; Spice_Lib_File (none) -> spice_components.lib; Spice_Model (none) -> bd135; Spice_Netlist_Enabled (none) -> Y; Spice_Primitive (none) -> Q
- Q2: renamed from Q?; Spice_Lib_File (none) -> spice_components.lib; Spice_Model (none) -> bd136; Spice_Netlist_Enabled (none) -> Y; Spice_Primitive (none) -> Q
- R3, R4: renamed from R?; value R -> 1k
- R5: renamed from R?; value R -> 10k
- R6: renamed from R?; value R -> 25; Spice_Model (none) -> 25; Spice_Netlist_Enabled (none) -> Y; Spice_Primitive (none) -> R
- U1: renamed from U?; symbol Amplifier_Operational:TL081 -> classAB_simul-rescue:TL081-RESCUE-classAB_simul; Spice_Lib_File (none) -> spice_components.lib; Spice_Model (none) -> TL081; Spice_Netlist_Enabled (none) -> Y; Spice_Node_Sequence (none) -> 3 2 7 4 6; Spice_Primitive (none) -> X
- V1: renamed from V?; Spice_Model (none) -> dc 12; Spice_Netlist_Enabled (none) -> Y; Spice_Primitive (none) -> V
- V2: renamed from V?; Spice_Model (none) -> dc 1 ac 1 sin(0 800m 5k); Spice_Netlist_Enabled (none) -> Y; Spice_Primitive (none) -> V
- gave numbers to parts that had none: 2
Connections:
- net labels added: DRIVE, IN, N_GATE, OUT, P_GATE
- wire segments 44 -> 46
Other:
- note added: "measurement resistor\n"

Commit message: update simulation, basically sorted
Parts:
- added R7: 25, symbol pspice:R
- 50u1: renamed from 230u1; Spice_Model 230u -> 50u; Spice_Netlist_Enabled Y -> N
- D1, D2: value 1N4148 -> DIODE; Spice_Node_Sequence (none) -> 2 1
- R5: value 10k -> 1k
Connections:
- wire segments 46 -> 47
Changed lines of the file:
@@
 $EndComp
-Wire Wire Line
-	6475 2000 6475 2350
 Wire Wire Line
 	5250 2700 6025 2700
@@
 P 5250 2150
 F 0 "R5" H 5318 2196 50  0000 L CNN
-F 1 "10k" H 5318 2105 50  0000 L CNN
+F 1 "1k" H 5318 2105 50  0000 L CNN
 F 2 "" H 5250 2150 50  0001 C CNN
 F 3 "" H 5250 2150 50  0001 C CNN
@@
 	1    0    0    -1
 $EndComp
-Wire Wire Line
-	5250 2400 5250 2700
-Connection ~ 5250 2700
 $Comp
 L power:VDD #PWR03
@@
 L pspice:R R6
 U 1 1 5A6625E0
-P 9275 4350
-F 0 "R6" H 9343 4396 50  0000 L CNN
-F 1 "25" H 9343 4305 50  0000 L CNN
-F 2 "" H 9275 4350 50  0001 C CNN
-F 3 "" H 9275 4350 50  0001 C CNN
-F 4 "R" H 9275 4350 60  0001 C CNN "Spice_Primitive"
-F 5 "25" H 9275 4350 60  0001 C CNN "Spice_Model"
-F 6 "Y" H 9275 4350 60  0001 C CNN "Spice_Netlist_Enabled"
-	1    9275 4350
+P 9275 3950
+F 0 "R6" H 9343 3996 50  0000 L CNN
+F 1 "25" H 9343 3905 50  0000 L CNN
+F 2 "" H 9275 3950 50  0001 C CNN
+F 3 "" H 9275 3950 50  0001 C CNN
+F 4 "R" H 9275 3950 60  0001 C CNN "Spice_Primitive"
+F 5 "25" H 9275 3950 60  0001 C CNN "Spice_Model"
+F 6 "Y" H 9275 3950 60  0001 C CNN "Spice_Netlist_Enabled"
+	1    9275 3950
 	1    0    0    -1
 $EndComp
@@
 	1    0    0    -1
 $EndComp
-Wire Wire Line
-	9275 5175 9275 4850
-Wire Wire Line
-	9275 4100 9275 3850
 Connection ~ 6475 3400
 Wire Wire Line
@@
 	1875 2450 1875 2550
 $Comp
-L pspice:INDUCTOR 230u1
+L pspice:INDUCTOR 50u1
 U 1 1 5A666D29
-P 9950 4350
-F 0 "230u1" V 9904 4428 50  0000 L CNN
-F 1 "INDUCTOR" V 9995 4428 50  0000 L CNN
-F 2 "" H 9950 4350 50  0001 C CNN
-F 3 "" H 9950 4350 50  0001 C CNN
-F 4 "L" H 9950 4350 60  0001 C CNN "Spice_Primitive"
-F 5 "230u" H 9950 4350 60  0001 C CNN "Spice_Model"
-F 6 "Y" H 9950 4350 60  0001 C CNN "Spice_Netlist_Enabled"
-	1    9950 4350
-	0    1    1    0
-$EndComp
-Wire Wire Line
-	9950 4600 9950 4850
-Wire Wire Line
-	9950 4850 9275 4850
-Connection ~ 9275 4850
-Wire Wire Line
-	9275 4850 9275 4600
-Wire Wire Line
-	9950 4100 9950 3850
-Wire Wire Line
-	9950 3850 9275 3850
-Connection ~ 9275 3850
-Wire Wire Line
-	9275 3850 9275 3400
+P 9275 4575
+F 0 "50u1" V 9229 4653 50  0000 L CNN
+F 1 "INDUCTOR" V 9320 4653 50  0000 L CNN
+F 2 "" H 9275 4575 50  0001 C CNN
+F 3 "" H 9275 4575 50  0001 C CNN
+F 4 "L" H 9275 4575 60  0001 C CNN "Spice_Primitive"
+F 5 "50u" H 9275 4575 60  0001 C CNN "Spice_Model"
+F 6 "N" H 9275 4575 60  0001 C CNN "Spice_Netlist_Enabled"
+	1    9275 4575
+	0    1    1    0
+$EndComp
 Wire Notes Line
 	8675 3650 10950 3650
@@
 Text Label 5600 4200 0    60   ~ 0
 P_GATE
-$Comp
-L pspice:DIODE D1
-U 1 1 5A66A983
-P 5250 3200
-F 0 "D1" V 5204 3328 50  0000 L CNN
-F 1 "1N4148" V 5295 3328 50  0000 L CNN
-F 2 "" H 5250 3200 50  0001 C CNN
-F 3 "" H 5250 3200 50  0001 C CNN
-F 4 "X" H 5250 3200 60  0001 C CNN "Spice_Primitive"
-F 5 "1N4148" H 5250 3200 60  0001 C CNN "Spice_Model"
-F 6 "Y" H 5250 3200 60  0001 C CNN "Spice_Netlist_Enabled"
-F 7 "spice_components.lib" H 5250 3200 60  0001 C CNN "Spice_Lib_File"
-	1    5250 3200
-	0    1    1    0
-$EndComp
-Wire Wire Line
-	5250 2700 5250 3000
 Wire Wire Line
 	7250 775  7250 850
@@
 Text Notes 7550 725  0    60   ~ 0
 measurement resistor\n
+Connection ~ 3300 4300
+Wire Wire Line
+	3100 4300 3300 4300
+Wire Wire Line
+	2275 4300 2600 4300
+Wire Wire Line
+	7250 850  8250 850
+Wire Wire Line
+	5250 2400 5250 2700
+$Comp
+L pspice:DIODE D1
+U 1 1 5A682A3B
+P 5250 3050
+F 0 "D1" V 5204 3178 50  0000 L CNN
+F 1 "DIODE" V 5295 3178 50  0000 L CNN
+F 2 "" H 5250 3050 50  0001 C CNN
+F 3 "" H 5250 3050 50  0001 C CNN
+F 4 "X" H 5250 3050 60  0001 C CNN "Spice_Primitive"
+F 5 "1N4148" H 5250 3050 60  0001 C CNN "Spice_Model"
+F 6 "Y" H 5250 3050 60  0001 C CNN "Spice_Netlist_Enabled"
+F 7 "spice_components.lib" H 5250 3050 60  0001 C CNN "Spice_Lib_File"
+F 8 "2 1" H 5250 3050 60  0001 C CNN "Spice_Node_Sequence"
+	1    5250 3050
+	0    1    1    0
+$EndComp
 $Comp
 L pspice:DIODE D2
-U 1 1 5A66FB13
-P 5250 3750
-F 0 "D2" V 5204 3878 50  0000 L CNN
-F 1 "1N4148" V 5295 3878 50  0000 L CNN
-F 2 "" H 5250 3750 50  0001 C CNN
-F 3 "" H 5250 3750 50  0001 C CNN
-F 4 "X" H 5250 3750 60  0001 C CNN "Spice_Primitive"
-F 5 "1N4148" H 5250 3750 60  0001 C CNN "Spice_Model"
-F 6 "Y" H 5250 3750 60  0001 C CNN "Spice_Netlist_Enabled"
-F 7 "spice_components.lib" H 5250 3750 60  0001 C CNN "Spice_Lib_File"
-	1    5250 3750
-	0    1    1    0
-$EndComp
-Wire Wire Line
-	5250 3400 5250 3550
+U 1 1 5A682AE7
+P 5250 3625
+F 0 "D2" V 5204 3753 50  0000 L CNN
+F 1 "DIODE" V 5295 3753 50  0000 L CNN
+F 2 "" H 5250 3625 50  0001 C CNN
+F 3 "" H 5250 3625 50  0001 C CNN
+F 4 "X" H 5250 3625 60  0001 C CNN "Spice_Primitive"
+F 5 "1N4148" H 5250 3625 60  0001 C CNN "Spice_Model"
+F 6 "Y" H 5250 3625 60  0001 C CNN "Spice_Netlist_Enabled"
+F 7 "spice_components.lib" H 5250 3625 60  0001 C CNN "Spice_Lib_File"
+F 8 "2 1" H 5250 3625 60  0001 C CNN "Spice_Node_Sequence"
+	1    5250 3625
+	0    1    1    0
+$EndComp
+Wire Wire Line
+	5250 2850 5250 2700
+Connection ~ 5250 2700
+Wire Wire Line
+	5250 3825 5250 4200
+Wire Wire Line
+	5250 4200 6025 4200
+Wire Wire Line
+	5250 3250 5250 3425
+Connection ~ 5250 4200
+Wire Wire Line
+	9275 4200 9275 4250
+$Comp
+L pspice:R R7
+U 1 1 5A68AF3A
+P 10150 4575
+F 0 "R7" H 10218 4621 50  0000 L CNN
+F 1 "25" H 10218 4530 50  0000 L CNN
+F 2 "" H 10150 4575 50  0001 C CNN
+F 3 "" H 10150 4575 50  0001 C CNN
+F 4 "R" H 10150 4575 60  0001 C CNN "Spice_Primitive"
+F 5 "10k" H 10150 4575 60  0001 C CNN "Spice_Model"
+F 6 "Y" H 10150 4575 60  0001 C CNN "Spice_Netlist_Enabled"
+	1    10150 4575
+	1    0    0    -1
+$EndComp
+Wire Wire Line
+	10150 4325 10150 4250
+Wire Wire Line
+	10150 4250 9275 4250
+Wire Wire Line
+	9275 3400 9275 3700
+Wire Wire Line
+	9275 4825 9275 4975
+Connection ~ 9275 4250
+Wire Wire Line
+	9275 4250 9275 4325
+Wire Wire Line
+	10150 4825 10150 4975
+Wire Wire Line
+	10150 4975 9275 4975
+Connection ~ 9275 4975
+Wire Wire Line
+	9275 4975 9275 5175
+Wire Wire Line
+	6475 2000 6475 2350
+Wire Wire Line
+	8550 3400 9275 3400
+Wire Wire Line
+	7750 3400 8050 3400
+Wire Wire Line
+	975  4300 1775 4300
 Wire Wire Line
 	4125 4200 5250 4200
-Wire Wire Line
-	5250 3950 5250 4200
-Connection ~ 5250 4200
-Wire Wire Line
-	5250 4200 6025 4200
-Connection ~ 3300 4300
-Wire Wire Line
-	3100 4300 3300 4300
-Wire Wire Line
-	8550 3400 9275 3400
-Wire Wire Line
-	7750 3400 8050 3400
-Wire Wire Line
-	2275 4300 2600 4300
-Wire Wire Line
-	975  4300 1775 4300
-Wire Wire Line
-	7250 850  8250 850
 $EndSCHEMATC
